File: hw/can_gauge_interface.kicad_sch (KiCad schematic)
At the start: 56 parts, among them U1 MCP2515-I/P, U2 AP64100Q, U3 MCP2561-E-P, U4 25LC160C, U5 PIC16F1459-IP, U6 MCP4912

Commit message: hw: 6v6 debug pin
Parts:
- added J?: Conn_01x01_Socket, symbol Connector:Conn_01x01_Socket
Connections:
- net +5VA is gone; now on net +5V: C8.1, C?.1, C?.1, J?.1 (Pin_1), R4.1, R?.1, U6.1 (Vdd), U6.11 (VrefB), U6.13 (VrefA), U6.9 (~{SHDN}), U?.1 (VO), U?.1 (Vdd), U?.11 (VrefB), U?.13 (VrefA), U?.9 (~{SHDN})
Other:
- moved on the sheet: C?, H1, H2, H3, H4, J?, JP?, R?, U1, U3, U4

Commit message: hw: connected pic gpios
Parts:
- added JP4: USB_PWR, symbol Jumper:Jumper_2_Open
- gave numbers to parts that had none: 33
- renumbered C6 to C10, C7 to C11, C8 to C17, C4 to C3, C3 to C4, R4 to R11, U5 to U1, U1 to U2, U2 to U5, U6 to U9
Connections:
- net MCP2515_~{CS} is gone; now on net CAN_~{CS}: J5.4 (Pin_4), R7.2, U2.16 (~{CS})
- net +5V: no longer C16.1, C17.1, C9.1, J9.1 (Pin_1), R10.1, R11.1, U7.1 (VO), U8.1 (Vdd), U8.11 (VrefB), U8.13 (VrefA), U8.9 (~{SHDN}), U9.1 (Vdd), U9.11 (VrefB), U9.13 (VrefA), U9.9 (~{SHDN})
- net DAC1_~{CS}: now also U1.10 (RB7/TX/CK)
- net DAC2_~{CS}: now also U1.14 (C2IN2-/C1IN2-/DACOUT1/AN6/RC2)
- net GND: now also U3.8 (STBY)
- net Speed: now also U1.6 (CWG1B/C1OUT/C2OUT/RC4)
- net Tach: now also U1.7 (CLKR/C1IN3-/C2IN3-/DACOUT2/AN7/RC3)
- net VBUS: now also JP4.1 (A)
- net CAN_~{CS}: now reaches U1.12 (RB5/AN11/RX/DX)
- new net +5VA: C16.1, C17.1, C9.1, J9.1 (Pin_1), JP4.2 (B), R10.1, R11.1, U7.1 (VO), U8.1 (Vdd), U8.11 (VrefB), U8.13 (VrefA), U8.9 (~{SHDN}), U9.1 (Vdd), U9.11 (VrefB), U9.13 (VrefA), U9.9 (~{SHDN})
- no-connect marks 6 -> 8
Other:
- moved on the sheet: J1, J2, J3, JP3

Commit message: hw: fixed erc warnings
Parts:
- removed U2: MCP2515-I/P, Package_SO:SOIC-18W_7.5x11.6mm_P1.27mm, symbol Interface_CAN_LIN:MCP2515-xSO
- added U2: MCP2515-I/P, Package_DIP:DIP-18_W7.62mm, symbol symbols:MCP2515-I/P
Connections:
- net +5V: now also U2.17 (~{RESET}), U2.18 (VDD), U2.4 (~{TX0RTS}), U2.5 (~{TX1RTS}), U2.6 (~{TX2RTS})
- net CAN_~{CS}: now also U2.16 (~{CS})
- net CLK: now also U2.8 (OSC1)
- net GND: now also U2.9 (VSS)
- net INT: now also U2.12 (~{INT})
- net MISO: now also U2.15 (SO)
- net MOSI: now also U2.14 (SI)
- net SCK: now also U2.13 (SCK)
- net +6.5V: now reaches C2.2, C3.2, C6.1, L1.2, R1.2, U6.7 (EN), U6.8 (VI)
- net +6.5V: now also C8.1, J7.1 (Pin_1), U7.7 (EN), U7.8 (VI)
- net at U3.1 (TXD): now also U2.1 (TXCAN)
- net at U3.4 (RXD): now also U2.2 (RXCAN)

Commit message: footprints
Parts:
- C1, C10, C12, C13, C14, C15, C16, C17, C2, C3, C4, C6, C7, C8, C9: footprint (none) -> Capacitor_SMD:C_1206_3216Metric_Pad1.33x1.80mm_HandSolder
- C11: value 470n -> 1u; footprint (none) -> Capacitor_SMD:C_1206_3216Metric_Pad1.33x1.80mm_HandSolder
- C5: value 58n -> 100n; footprint (none) -> Capacitor_SMD:C_1206_3216Metric_Pad1.33x1.80mm_HandSolder
- J1: footprint (none) -> Connector_USB:USB_A_Wuerth_614004134726_Horizontal
- J10, J6, J7, J8, J9: footprint (none) -> Connector_PinSocket_2.54mm:PinSocket_1x01_P2.54mm_Vertical
- J3: footprint (none) -> Connector_Molex:Molex_Mini-Fit_Jr_5569-06A2_2x03_P4.20mm_Horizontal
- J4: footprint (none) -> Connector_PinHeader_2.54mm:PinHeader_1x05_P2.54mm_Vertical
- J5: footprint (none) -> Connector_PinSocket_2.54mm:PinSocket_1x07_P2.54mm_Vertical
- JP1, JP3, JP4, JP5: footprint (none) -> Connector_PinSocket_2.54mm:PinSocket_1x02_P2.54mm_Vertical
- JP2: footprint (none) -> Connector_PinSocket_2.54mm:PinSocket_1x03_P2.54mm_Vertical
- L1: footprint (none) -> Inductor_SMD:L_Wuerth_WE-PD-Typ-LS_Handsoldering
- R1: value 72k5 -> 73k2; footprint (none) -> Resistor_SMD:R_0805_2012Metric_Pad1.20x1.40mm_HandSolder
- R10, R11, R2, R3, R4, R6, R7, R8, R9: footprint (none) -> Resistor_SMD:R_0805_2012Metric_Pad1.20x1.40mm_HandSolder
- R5: value 10k -> 12k; footprint (none) -> Resistor_SMD:R_0805_2012Metric_Pad1.20x1.40mm_HandSolder
- U1: footprint (none) -> Package_DIP:DIP-20_W7.62mm
- U4: footprint (none) -> Package_DIP:DIP-8-16_W7.62mm
- U8, U9: footprint (none) -> Package_DIP:DIP-14_W7.62mm
Other:
- note added: "6.7V R±1%"
- note removed: "6.5V R±1%"
- company: (none) -> Sam Anthony
- title: (none) -> CAN Gauge Interface
Changed lines of the file:
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@@
 	(generator_version "9.0")
 	(paper "A2")
+	(title_block
+		(title "CAN Gauge Interface")
+		(date "2025-09-19")
+		(rev "0.1")
+		(company "Sam Anthony")
+	)
 	(rectangle
 		(start 482.6 41.91)
@@
 		)
 	)
-	(text "6.5V\nR±1%"
+	(text "6.7V\nR±1%"
 		(exclude_from_sim no)
 		(at 95.25 69.85 0)
@@
 			)
 		)
-		(property "Footprint" ""
+		(property "Footprint" "Connector_USB:USB_A_Wuerth_614004134726_Horizontal"
 			(at 44.45 154.94 0)
 			(effects
@@
 			)
 		)
-		(property "Footprint" ""
+		(property "Footprint" "Capacitor_SMD:C_1206_3216Metric_Pad1.33x1.80mm_HandSolder"
 			(at 174.9552 60.96 0)
 			(effects
@@
 			)
 		)
-		(property "Footprint" ""
+		(property "Footprint" "Capacitor_SMD:C_1206_3216Metric_Pad1.33x1.80mm_HandSolder"
 			(at 133.35 151.4348 0)
 			(effects
@@
 			)
 		)
-		(property "Footprint" ""
+		(property "Footprint" "Connector_PinSocket_2.54mm:PinSocket_1x02_P2.54mm_Vertical"
 			(at 240.03 76.2 0)
 			(effects
@@
 			)
 		)
-		(property "Footprint" ""
+		(property "Footprint" "Capacitor_SMD:C_1206_3216Metric_Pad1.33x1.80mm_HandSolder"
 			(at 270.51 148.8948 0)
 			(effects
@@
 			)
 		)
-		(property "Footprint" ""
+		(property "Footprint" "Capacitor_SMD:C_1206_3216Metric_Pad1.33x1.80mm_HandSolder"
 			(at 105.7148 53.34 0)
 			(effects
@@
 			)
 		)
-		(property "Footprint" ""
+		(property "Footprint" "Capacitor_SMD:C_1206_3216Metric_Pad1.33x1.80mm_HandSolder"
 			(at 31.4452 52.07 0)
 			(effects
@@
 			)
 		)
-		(property "Footprint" ""
+		(property "Footprint" "Capacitor_SMD:C_1206_3216Metric_Pad1.33x1.80mm_HandSolder"
 			(at 496.2652 67.31 0)
 			(effects
@@
 			)
 		)
-		(property "Footprint" ""
+		(property "Footprint" "Package_DIP:DIP-8-16_W7.62mm"
 			(at 137.16 167.64 0)
 			(effects
@@
 			)
 		)
-		(property "Footprint" ""
+		(property "Footprint" "Connector_PinSocket_2.54mm:PinSocket_1x03_P2.54mm_Vertical"
 			(at 403.86 64.77 0)
 			(effects
@@
 			)
 		)
-		(property "Footprint" ""
+		(property "Footprint" "Resistor_SMD:R_0805_2012Metric_Pad1.20x1.40mm_HandSolder"
 			(at 199.136 153.924 90)
 			(effects
@@
 			)
 		)
-		(property "Footprint" ""
+		(property "Footprint" "Resistor_SMD:R_0805_2012Metric_Pad1.20x1.40mm_HandSolder"
 			(at 119.126 164.084 90)
 			(effects
@@
 			)
 		)
-		(property "Footprint" ""
+		(property "Footprint" "Connector_PinSocket_2.54mm:PinSocket_1x07_P2.54mm_Vertical"
 			(at 38.1 243.84 0)
 			(effects
@@
 			)
 		)
-		(property "Footprint" ""
+		(property "Footprint" "Connector_PinSocket_2.54mm:PinSocket_1x02_P2.54mm_Vertical"
 			(at 62.23 143.51 0)
 			(effects
@@
 			)
 		)
-		(property "Footprint" ""
+		(property "Footprint" "Capacitor_SMD:C_1206_3216Metric_Pad1.33x1.80mm_HandSolder"
 			(at 144.4752 60.96 0)
 			(effects
@@
 			)
 		)
-		(property "Footprint" ""
+		(property "Footprint" "Connector_PinSocket_2.54mm:PinSocket_1x02_P2.54mm_Vertical"
 			(at 62.23 148.59 0)
 			(effects
@@
 			)
 		)
-		(property "Footprint" ""
+		(property "Footprint" "Capacitor_SMD:C_1206_3216Metric_Pad1.33x1.80mm_HandSolder"
 			(at 205.74 141.2748 0)
 			(effects
@@
 			)
 		)
-		(property "Value" "10k"
+		(property "Value" "12k"
 			(at 73.66 59.69 0)
 			(effects
@@
 			)
 		)
-		(property "Footprint" ""
+		(property "Footprint" "Resistor_SMD:R_0805_2012Metric_Pad1.20x1.40mm_HandSolder"
 			(at 68.834 58.166 90)
 			(effects
@@
 			)
 		)
-		(property "Footprint" ""
+		(property "Footprint" "Capacitor_SMD:C_1206_3216Metric_Pad1.33x1.80mm_HandSolder"
 			(at 521.6652 67.31 0)
 			(effects
@@
 			)
 		)
-		(property "Footprint" ""
+		(property "Footprint" "Resistor_SMD:R_0805_2012Metric_Pad1.20x1.40mm_HandSolder"
 			(at 40.386 59.944 90)
 			(effects
@@
 			)
 		)
-		(property "Footprint" ""
+		(property "Footprint" "Capacitor_SMD:C_1206_3216Metric_Pad1.33x1.80mm_HandSolder"
 			(at 240.9952 91.44 0)
 			(effects
@@
 			)
 		)
-		(property "Footprint" ""
+		(property "Footprint" "Resistor_SMD:R_0805_2012Metric_Pad1.20x1.40mm_HandSolder"
 			(at 91.694 61.976 90)
 			(effects
@@
 			)
 		)
-		(property "Footprint" ""
+		(property "Footprint" "Capacitor_SMD:C_1206_3216Metric_Pad1.33x1.80mm_HandSolder"
 			(at 525.78 162.8648 0)
 			(effects
@@
 			)
 		)
-		(property "Footprint" ""
+		(property "Footprint" "Package_DIP:DIP-14_W7.62mm"
 			(at 530.86 124.46 0)
 			(effects
@@
 			)
 		)
-		(property "Footprint" ""
+		(property "Footprint" "Resistor_SMD:R_0805_2012Metric_Pad1.20x1.40mm_HandSolder"
 			(at 250.444 66.294 90)
 			(effects
@@
 			)
 		)
-		(property "Footprint" ""
+		(property "Footprint" "Connector_PinSocket_2.54mm:PinSocket_1x01_P2.54mm_Vertical"
 			(at 38.1 266.7 0)
 			(effects
@@
 			)
 		)
-		(property "Footprint" ""
+		(property "Footprint" "Connector_PinSocket_2.54mm:PinSocket_1x01_P2.54mm_Vertical"
 			(at 38.1 293.37 0)
 			(effects
@@
 			)
 		)
-		(property "Footprint" ""
+		(property "Footprint" "Capacitor_SMD:C_1206_3216Metric_Pad1.33x1.80mm_HandSolder"
 			(at 69.85 42.8752 0)
 			(effects
@@
 			)
 		)
-		(property "Footprint" ""
+		(property "Footprint" "Connector_Molex:Molex_Mini-Fit_Jr_5569-06A2_2x03_P4.20mm_Horizontal"
 			(at 49.53 209.55 0)
 			(effects
@@
 			)
 		)
-		(property "Footprint" ""
+		(property "Footprint" "Connector_PinSocket_2.54mm:PinSocket_1x01_P2.54mm_Vertical"
 			(at 38.1 275.59 0)
 			(effects
@@
 			)
 		)
-		(property "Footprint" ""
+		(property "Footprint" "Connector_PinSocket_2.54mm:PinSocket_1x01_P2.54mm_Vertical"
 			(at 38.1 302.26 0)
 			(effects
@@
 			)
 		)
-		(property "Footprint" ""
+		(property "Footprint" "Resistor_SMD:R_0805_2012Metric_Pad1.20x1.40mm_HandSolder"
 			(at 241.046 59.944 90)
 			(effects
@@
 			)
 		)
-		(property "Footprint" ""
+		(property "Footprint" "Capacitor_SMD:C_1206_3216Metric_Pad1.33x1.80mm_HandSolder"
 			(at 323.85 46.6852 0)
 			(effects
@@
 			)
 		)
-		(property "Footprint" ""
+		(property "Footprint" "Connector_PinHeader_2.54mm:PinHeader_1x05_P2.54mm_Vertical"
 			(at 38.1 119.38 0)
 			(effects
@@
 			)
 		)
-		(property "Value" "58n"
+		(property "Value" "100n"
 			(at 74.93 67.945 0)
 			(effects
@@
 			)
 		)
-		(property "Footprint" ""
+		(property "Footprint" "Capacitor_SMD:C_1206_3216Metric_Pad1.33x1.80mm_HandSolder"
 			(at 68.8848 63.5 0)
 			(effects
@@
 			)
 		)
-		(property "Footprint" ""
+		(property "Footprint" "Connector_PinSocket_2.54mm:PinSocket_1x02_P2.54mm_Vertical"
 			(at 299.72 157.48 0)
 			(effects
@@
 			)
 		)
-		(property "Footprint" ""
+		(property "Footprint" "Capacitor_SMD:C_1206_3216Metric_Pad1.33x1.80mm_HandSolder"
 			(at 525.78 99.3648 0)
 			(effects
@@
 			)
 		)
-		(property "Footprint" ""
+		(property "Footprint" "Capacitor_SMD:C_1206_3216Metric_Pad1.33x1.80mm_HandSolder"
 			(at 115.8748 53.34 0)
 			(effects
@@
 			)
 		)
-		(property "Footprint" ""
+		(property "Footprint" "Package_DIP:DIP-14_W7.62mm"
 			(at 530.86 187.96 0)
 			(effects
@@
 			)
 		)
-		(property "Footprint" ""
+		(property "Footprint" "Resistor_SMD:R_0805_2012Metric_Pad1.20x1.40mm_HandSolder"
 			(at 489.966 109.474 90)
 			(effects
@@
 			)
 		)
-		(property "Value" "72k5"
+		(property "Value" "73k2"
 			(at 97.155 53.975 0)
 			(effects
@@
 			)
 		)
-		(property "Footprint" ""
+		(property "Footprint" "Resistor_SMD:R_0805_2012Metric_Pad1.20x1.40mm_HandSolder"
 			(at 91.694 51.816 90)
 			(effects
@@
 		(dnp no)
 		(property "Reference" "C11"
-			(at 271.78 46.355 90)
+			(at 274.32 46.355 90)
 			(effects
 				(font
@@
 			)
 		)
-		(property "Value" "470n"
-			(at 270.51 48.895 90)
+		(property "Value" "1u"
+			(at 271.145 48.26 90)
 			(effects
 				(font
@@
 			)
 		)
-		(property "Footprint" ""
+		(property "Footprint" "Capacitor_SMD:C_1206_3216Metric_Pad1.33x1.80mm_HandSolder"
 			(at 270.51 51.7652 0)
 			(effects
@@
 			)
 		)
-		(property "Footprint" ""
+		(property "Footprint" "Package_DIP:DIP-20_W7.62mm"
 			(at 334.01 67.31 0)
 			(effects
@@
 			)
 		)
-		(property "Footprint" ""
+		(property "Footprint" "Resistor_SMD:R_0805_2012Metric_Pad1.20x1.40mm_HandSolder"
 			(at 489.966 172.974 90)
 			(effects
@@
 			)
 		)
-		(property "Footprint" ""
+		(property "Footprint" "Connector_PinSocket_2.54mm:PinSocket_1x01_P2.54mm_Vertical"
 			(at 38.1 284.48 0)
 			(effects
@@
 			)
 		)
-		(property "Footprint" ""
+		(property "Footprint" "Resistor_SMD:R_0805_2012Metric_Pad1.20x1.40mm_HandSolder"
 			(at 310.134 156.464 90)
 			(effects
@@
 			)
 		)
-		(property "Footprint" ""
+		(property "Footprint" "Inductor_SMD:L_Wuerth_WE-PD-Typ-LS_Handsoldering"
 			(at 86.36 45.72 0)
 			(effects

Commit message: buck converter layout and routing
Parts:
- J1: footprint Connector_USB:USB_A_Wuerth_614004134726_Horizontal -> Connector_USB:USB_B_OST_USB-B1HSxx_Horizontal
- U4: footprint Package_DIP:DIP-8-16_W7.62mm -> Package_DIP:DIP-8_W7.62mm
Connections:
- net GND: now also U5.9 (EP), U6.5 (GND), U6.9 (EP), U7.5 (GND), U7.9 (EP); no longer U6.3 (GND), U7.3 (GND)
Changed lines of the file:
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@@
 	)
 	(junction
+		(at 158.75 58.42)
+		(diameter 0)
+		(color 0 0 0 0)
+	)
+	(junction
 		(at 510.54 166.37)
 		(diameter 0)
@@
 	)
 	(junction
+		(at 504.19 68.58)
+		(diameter 0)
+		(color 0 0 0 0)
+	)
+	(junction
 		(at 106.68 45.72)
 		(diameter 0)
@@
 	)
 	(junction
+		(at 55.88 64.77)
+		(diameter 0)
+		(color 0 0 0 0)
+	)
+	(junction
 		(at 525.78 175.26)
 		(diameter 0)
@@
 	(wire
 		(pts
+			(xy 158.75 58.42) (xy 158.75 73.66)
+		)
+		(stroke
+			(width 0)
+			(type default)
+		)
+	)
+	(wire
+		(pts
 			(xy 495.3 182.88) (xy 497.84 182.88)
 		)
@@
 	(wire
 		(pts
+			(xy 154.94 55.88) (xy 154.94 58.42)
+		)
+		(stroke
+			(width 0)
+			(type default)
+		)
+	)
+	(wire
+		(pts
 			(xy 497.84 111.76) (xy 496.57 111.76)
 		)
@@
 	(wire
 		(pts
+			(xy 49.53 62.23) (xy 49.53 64.77)
+		)
+		(stroke
+			(width 0)
+			(type default)
+		)
+	)
+	(wire
+		(pts
 			(xy 525.78 168.91) (xy 525.78 175.26)
 		)
@@
 	(wire
 		(pts
-			(xy 55.88 62.23) (xy 55.88 73.66)
+			(xy 55.88 62.23) (xy 55.88 64.77)
 		)
 		(stroke
@@
 	(wire
 		(pts
+			(xy 154.94 58.42) (xy 158.75 58.42)
+		)
+		(stroke
+			(width 0)
+			(type default)
+		)
+	)
+	(wire
+		(pts
 			(xy 44.45 180.34) (xy 40.64 180.34)
 		)
@@
 	(wire
 		(pts
+			(xy 504.19 68.58) (xy 508 68.58)
+		)
+		(stroke
+			(width 0)
+			(type default)
+		)
+	)
+	(wire
+		(pts
 			(xy 233.68 152.4) (xy 215.9 152.4)
 		)
@@
 	(wire
 		(pts
-			(xy 158.75 55.88) (xy 158.75 73.66)
+			(xy 158.75 55.88) (xy 158.75 58.42)
 		)
 		(stroke
@@
 	(wire
 		(pts
-			(xy 495.3 68.58) (xy 508 68.58)
+			(xy 495.3 68.58) (xy 504.19 68.58)
 		)
 		(stroke
@@
 	(wire
 		(pts
+			(xy 49.53 64.77) (xy 55.88 64.77)
+		)
+		(stroke
+			(width 0)
+			(type default)
+		)
+	)
+	(wire
+		(pts
 			(xy 215.9 138.43) (xy 215.9 142.24)
 		)
@@
 	(wire
 		(pts
+			(xy 504.19 67.31) (xy 504.19 68.58)
+		)
+		(stroke
+			(width 0)
+			(type default)
+		)
+	)
+	(wire
+		(pts
 			(xy 86.36 57.15) (xy 86.36 49.53)
 		)
@@
 	(wire
 		(pts
+			(xy 55.88 64.77) (xy 55.88 73.66)
+		)
+		(stroke
+			(width 0)
+			(type default)
+		)
+	)
+	(wire
+		(pts
 			(xy 182.88 162.56) (xy 200.66 162.56)
 		)
@@
 			)
 		)
-		(property "Footprint" "Connector_USB:USB_A_Wuerth_614004134726_Horizontal"
+		(property "Footprint" "Connector_USB:USB_B_OST_USB-B1HSxx_Horizontal"
 			(at 44.45 154.94 0)
 			(effects
@@
 			)
 		)
-		(property "Footprint" "Package_DIP:DIP-8-16_W7.62mm"
+		(property "Footprint" "Package_DIP:DIP-8_W7.62mm"
 			(at 137.16 167.64 0)
 			(effects
@@
 		(pin "8"
 		)
+		(pin "9"
+		)
 		(instances
 			(project ""
@@
 		(pin "1"
 		)
+		(pin "4"
+		)
+		(pin "2"
+		)
+		(pin "6"
+		)
+		(pin "5"
+		)
+		(pin "9"
+		)
 		(instances
 			(project ""
@@
 	)
 	(symbol
+		(lib_name "AP7375Q_1")
 		(lib_id "symbols:AP7375Q")
 		(at 158.75 45.72 0)
@@
 		(pin "1"
 		)
+		(pin "2"
+		)
+		(pin "4"
+		)
+		(pin "6"
+		)
+		(pin "5"
+		)
+		(pin "9"
+		)
 		(instances

Commit message: analog routing
Connections:
- net AN3: now also J3.6 (Pin_6); no longer J3.3 (Pin_3)
- net AN4: now also J3.3 (Pin_3); no longer J3.6 (Pin_6)

Commit message: tht decoupling caps
Parts:
- C10, C12, C13, C14, C15, C16, C17, C4, C5: footprint Capacitor_SMD:C_1206_3216Metric_Pad1.33x1.80mm_HandSolder -> Capacitor_THT:C_Disc_D5.0mm_W2.5mm_P2.50mm
Changed lines of the file:
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@@
 			)
 		)
-		(property "Footprint" "Capacitor_SMD:C_1206_3216Metric_Pad1.33x1.80mm_HandSolder"
+		(property "Footprint" "Capacitor_THT:C_Disc_D5.0mm_W2.5mm_P2.50mm"
 			(at 133.35 151.4348 0)
 			(effects
@@
 			)
 		)
-		(property "Footprint" "Capacitor_SMD:C_1206_3216Metric_Pad1.33x1.80mm_HandSolder"
+		(property "Footprint" "Capacitor_THT:C_Disc_D5.0mm_W2.5mm_P2.50mm"
 			(at 270.51 148.8948 0)
 			(effects
@@
 			)
 		)
-		(property "Footprint" "Capacitor_SMD:C_1206_3216Metric_Pad1.33x1.80mm_HandSolder"
+		(property "Footprint" "Capacitor_THT:C_Disc_D5.0mm_W2.5mm_P2.50mm"
 			(at 205.74 141.2748 0)
 			(effects
@@
 			)
 		)
-		(property "Footprint" "Capacitor_SMD:C_1206_3216Metric_Pad1.33x1.80mm_HandSolder"
+		(property "Footprint" "Capacitor_THT:C_Disc_D5.0mm_W2.5mm_P2.50mm"
 			(at 240.9952 91.44 0)
 			(effects
@@
 			)
 		)
-		(property "Footprint" "Capacitor_SMD:C_1206_3216Metric_Pad1.33x1.80mm_HandSolder"
+		(property "Footprint" "Capacitor_THT:C_Disc_D5.0mm_W2.5mm_P2.50mm"
 			(at 525.78 162.8648 0)
 			(effects
@@
 			)
 		)
-		(property "Footprint" "Capacitor_SMD:C_1206_3216Metric_Pad1.33x1.80mm_HandSolder"
+		(property "Footprint" "Capacitor_THT:C_Disc_D5.0mm_W2.5mm_P2.50mm"
 			(at 69.85 42.8752 0)
 			(effects
@@
 			)
 		)
-		(property "Footprint" "Capacitor_SMD:C_1206_3216Metric_Pad1.33x1.80mm_HandSolder"
+		(property "Footprint" "Capacitor_THT:C_Disc_D5.0mm_W2.5mm_P2.50mm"
 			(at 323.85 46.6852 0)
 			(effects
@@
 			)
 		)
-		(property "Footprint" "Capacitor_SMD:C_1206_3216Metric_Pad1.33x1.80mm_HandSolder"
+		(property "Footprint" "Capacitor_THT:C_Disc_D5.0mm_W2.5mm_P2.50mm"
 			(at 68.8848 63.5 0)
 			(effects
@@
 			)
 		)
-		(property "Footprint" "Capacitor_SMD:C_1206_3216Metric_Pad1.33x1.80mm_HandSolder"
+		(property "Footprint" "Capacitor_THT:C_Disc_D5.0mm_W2.5mm_P2.50mm"
 			(at 525.78 99.3648 0)
 			(effects

Commit message: layout
Parts:
- R10, R11, R4, R6, R7, R9: footprint Resistor_SMD:R_0805_2012Metric_Pad1.20x1.40mm_HandSolder -> Resistor_THT:R_Axial_DIN0411_L9.9mm_D3.6mm_P12.70mm_Horizontal
Connections:
- net +12V: now also J2.4 (Pin_4); no longer J2.1 (Pin_1)
- net CAN_~{CS}: no longer U1.12 (RB5/AN11/RX/DX)
- net DAC1_~{CS}: no longer U1.10 (RB7/TX/CK)
- net DAC2_~{CS}: no longer U1.14 (C2IN2-/C1IN2-/DACOUT1/AN6/RC2)
- net GND: now also J2.8 (Pin_8); no longer J2.5 (Pin_5)
- net INT: now also JP2.1 (A); no longer JP2.2 (C)
- net ROM_~{CS}: no longer U1.2 (RA5/SOSCI/T1CKI/OSC1/CLKIN)
- net Speed: now also J2.5 (Pin_5); no longer J2.8 (Pin_8)
- net Tach: now also J2.1 (Pin_1); no longer J2.4 (Pin_4)
- net INT/ICSP_CLK: now reaches U1.15 (ICSPCLK/~{CWGFLT}/C2IN-/C1IN-/AN5/RC1)
- net INT/ICSP_CLK: now also JP2.2 (C); no longer JP2.1 (A)
- net CAN_TX: now reaches U2.1 (TXCAN), U3.1 (TXD)
- net CAN_RX: now reaches U2.2 (RXCAN), U3.4 (RXD)
Other:
- moved on the sheet: JP2
