File: hw/headers.kicad_sch (KiCad schematic)
At the start: 5 parts, among them J3 Power debug, J4 Power debug, J5 SPI debug, J6 I^{2}C debug, J7 CAN debug

Commit message: hw: erc: can
Connections:
- net FDCAN1.RX renamed CAN1.RX
- net FDCAN1.TX renamed CAN1.TX
Changed lines of the file:
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@@
 		)
 	)
-	(label "FDCAN1.RX"
+	(label "CAN1.RX"
 		(at 43.18 104.14 0)
 		(effects
@@
 		)
 	)
-	(label "FDCAN1.TX"
+	(label "CAN1.TX"
 		(at 43.18 101.6 0)
 		(effects
@@
 		)
 	)
-	(hierarchical_label "FDCAN1{CAN}"
+	(hierarchical_label "CAN1{CAN_IF}"
 		(shape input)
 		(at 63.5 99.06 0)
